Commit message: Created skeleton design for robot_control package

File: robot_description/urdf/basic_robot.urdf.xacro (robot description, xacro)
@@ -19,3 +19,18 @@
     </collision>
   </link>
+ <ros2_control name="GazeboSystem" type="system">
+  <hardware>
+    <plugin>gz_ros2_control/GazeboSystem</plugin>
+  </hardware>
+  <joint name="left_wheel_joint">
+    <command_interface name="velocity"/>
+    <state_interface name="position"/>
+    <state_interface name="velocity"/>
+  </joint>
+  <joint name="right_wheel_joint">
+    <command_interface name="velocity"/>
+    <state_interface name="position"/>
+    <state_interface name="velocity"/>
+  </joint>
+</ros2_control>
 </robot>
